File: qspimux-jspi1/qspimux-jspi1.kicad_pcb (KiCad board)
At the start: 2 copper layers, 49.5 x 20.3 mm, 8 parts, among them U1 TS3A27518E, U2 TS3A27518E, U3 W25Q128JVS

Commit message: wip
Parts:
- removed JEMU1: Conn_02x10_Counter_Clockwise, Connector_PinHeader_2.54mm:PinHeader_2x10_P2.54mm_Vertical
- removed JPROG1: Conn_02x07_Counter_Clockwise, Connector_PinHeader_2.54mm:PinHeader_2x07_P2.54mm_Vertical
- added JDEMU_1: Conn_JDEMU, Connector_PinHeader_2.54mm:PinHeader_2x05_P2.54mm_Vertical, F.Cu at (158.7, 109.2)
- added JDPRG100_1: Conn_JDPRG100, Connector_PinHeader_2.54mm:PinHeader_2x06_P2.54mm_Vertical, F.Cu at (153.7, 120.7)
- JSPI1: moved to B.Cu
- moved JSPI1 5.71 mm to (124.5, 117.5)
- moved U3 5.08 mm to (143.5, 114.3)
Other:
- board size 49.5 x 20.3 mm -> 41.9 x 20.3 mm
