File: qspimux-jspi1/qspimux-jspi1.kicad_sch (KiCad schematic)
At the start: 8 parts, among them U1 TS3A27518E, U2 TS3A27518E, U3 W25Q128JVS

Commit message: wip
Parts:
- removed JEMU1: Conn_02x10_Counter_Clockwise, Connector_PinHeader_2.54mm:PinHeader_2x10_P2.54mm_Vertical, symbol Connector_Generic:Conn_02x10_Counter_Clockwise
- removed JPROG1: Conn_02x07_Counter_Clockwise, Connector_PinHeader_2.54mm:PinHeader_2x07_P2.54mm_Vertical, symbol Connector_Generic:Conn_02x07_Counter_Clockwise
- added JDEMU_1: Conn_JDEMU, Connector_PinHeader_2.54mm:PinHeader_2x05_P2.54mm_Vertical, symbol common:Conn_JDEMU
- added JDPRG100_1: Conn_JDPRG100, Connector_PinHeader_2.54mm:PinHeader_2x06_P2.54mm_Vertical, symbol common:Conn_JDPRG100
